Commit message: Fix Gazebo vehicle colours

File: ros2_ws/src/ee5112_vehicle/urdf/vehicle.urdf.xacro (robot description, xacro)
@@ -54,5 +54,6 @@
   <xacro:property name="knuckle_mass" value="0.05"/>
   <!-- ========================================================= -->
-  <!-- MATERIALS                                                -->
+  <!-- MATERIALS (used by RViz - Gazebo needs its own tags,     -->
+  <!-- see the <gazebo reference="..."> blocks near the bottom) -->
   <!-- ========================================================= -->
   <material name="body_blue">
@@ -87,5 +88,5 @@
   <!-- ========================================================= -->
   <link name="base_link">
-    <visual name="chassis_visual">
+    <visual>
       <geometry>
         <box size="${chassis_length}
@@ -95,5 +96,5 @@
       <material name="body_blue"/>
     </visual>
-    <collision name="chassis_collision">
+    <collision>
       <geometry>
         <box size="${chassis_length}
@@ -316,5 +317,5 @@
   <!-- ========================================================= -->
   <link name="camera_link">
-    <visual name="camera_body">
+    <visual>
       <geometry>
         <box size="0.035 0.050 0.030"/>
@@ -322,5 +323,5 @@
       <material name="sensor_dark"/>
     </visual>
-    <visual name="camera_lens">
+    <visual>
       <origin
           xyz="0.0225 0 0"
@@ -333,5 +334,5 @@
       <material name="camera_lens_colour"/>
     </visual>
-    <collision name="camera_collision">
+    <collision>
       <geometry>
         <box size="0.035 0.050 0.030"/>
@@ -362,5 +363,5 @@
   <!-- ========================================================= -->
   <link name="laser_link">
-    <visual name="laser_body">
+    <visual>
       <geometry>
         <cylinder
@@ -370,5 +371,5 @@
       <material name="sensor_dark"/>
     </visual>
-    <visual name="laser_support">
+    <visual>
       <origin
           xyz="0 0 -0.035"
@@ -381,5 +382,5 @@
       <material name="steering_grey"/>
     </visual>
-    <collision name="laser_collision">
+    <collision>
       <geometry>
         <cylinder
@@ -409,7 +410,32 @@
   </joint>
   <!-- ========================================================= -->
-  <!-- GAZEBO WHEEL CONTACT                                     -->
-  <!-- ========================================================= -->
+  <!-- GAZEBO VISUAL MATERIALS                                  -->
+  <!-- ========================================================= -->
+  <!--
+       Gazebo classic's legacy URDF "gazebo extension" converter
+       expects <material> under <gazebo reference="..."> to be a
+       PLAIN TEXT built-in Ogre material script name (e.g.
+       "Gazebo/Blue"), not nested <ambient>/<diffuse> elements and
+       not wrapped in a named <visual> tag - both of those forms
+       were silently dropped, which is why the model kept
+       rendering grey. Each link below uses one of Gazebo's
+       built-in material names as the closest match to the
+       original custom RGBA colors.
+       Each link also gets exactly ONE <gazebo reference="...">
+       block (material + friction + sensor all merged together).
+       Multiple separate <gazebo reference> blocks for the same
+       link are not guaranteed to merge cleanly in Gazebo classic.
+  -->
+  <gazebo reference="base_link">
+    <material>Gazebo/Blue</material>
+  </gazebo>
+  <gazebo reference="front_left_steering_link">
+    <material>Gazebo/Grey</material>
+  </gazebo>
+  <gazebo reference="front_right_steering_link">
+    <material>Gazebo/Grey</material>
+  </gazebo>
   <gazebo reference="front_left_wheel_link">
+    <material>Gazebo/FlatBlack</material>
     <mu1>1.0</mu1>
     <mu2>1.0</mu2>
@@ -418,4 +444,5 @@
   </gazebo>
   <gazebo reference="front_right_wheel_link">
+    <material>Gazebo/FlatBlack</material>
     <mu1>1.0</mu1>
     <mu2>1.0</mu2>
@@ -424,4 +451,5 @@
   </gazebo>
   <gazebo reference="rear_left_wheel_link">
+    <material>Gazebo/FlatBlack</material>
     <mu1>1.0</mu1>
     <mu2>1.0</mu2>
@@ -430,4 +458,5 @@
   </gazebo>
   <gazebo reference="rear_right_wheel_link">
+    <material>Gazebo/FlatBlack</material>
     <mu1>1.0</mu1>
     <mu2>1.0</mu2>
@@ -436,11 +465,9 @@
   </gazebo>
   <!-- ========================================================= -->
-  <!-- GAZEBO RGB CAMERA                                        -->
-  <!-- ========================================================= -->
-  <!--
-       This is the already verified camera configuration.
-       Do not alter it while testing the LiDAR addition.
-  -->
+  <!-- GAZEBO RGB CAMERA (material + sensor merged into ONE      -->
+  <!-- <gazebo reference="camera_link"> block)                  -->
+  <!-- ========================================================= -->
   <gazebo reference="camera_link">
+    <material>Gazebo/DarkGrey</material>
     <sensor name="front_camera"
             type="camera">
@@ -485,4 +512,5 @@
   -->
   <gazebo reference="laser_link">
+    <material>Gazebo/DarkGrey</material>
     <sensor name="lidar"
             type="ray">

Commit message: Add Task 2 Ackermann trajectory validation

File: ros2_ws/src/ee5112_vehicle/urdf/vehicle.urdf.xacro (robot description, xacro)
@@ -54,6 +54,5 @@
   <xacro:property name="knuckle_mass" value="0.05"/>
   <!-- ========================================================= -->
-  <!-- MATERIALS (used by RViz - Gazebo needs its own tags,     -->
-  <!-- see the <gazebo reference="..."> blocks near the bottom) -->
+  <!-- MATERIALS                                                -->
   <!-- ========================================================= -->
   <material name="body_blue">
@@ -125,8 +124,10 @@
   <xacro:macro name="front_wheel"
                params="side x y">
+    <!-- Steering knuckle -->
     <link name="front_${side}_steering_link">
       <visual>
-        <origin xyz="0 0 0.025"
-                rpy="0 0 0"/>
+        <origin
+            xyz="0 0 0.025"
+            rpy="0 0 0"/>
         <geometry>
           <box size="0.025 0.025 0.070"/>
@@ -135,6 +136,7 @@
       </visual>
       <collision>
-        <origin xyz="0 0 0.025"
-                rpy="0 0 0"/>
+        <origin
+            xyz="0 0 0.025"
+            rpy="0 0 0"/>
         <geometry>
           <box size="0.025 0.025 0.070"/>
@@ -142,6 +144,7 @@
       </collision>
       <inertial>
-        <origin xyz="0 0 0.025"
-                rpy="0 0 0"/>
+        <origin
+            xyz="0 0 0.025"
+            rpy="0 0 0"/>
         <mass value="${knuckle_mass}"/>
         <inertia
@@ -223,6 +226,7 @@
       <parent link="front_${side}_steering_link"/>
       <child link="front_${side}_wheel_link"/>
-      <origin xyz="0 0 0"
-              rpy="0 0 0"/>
+      <origin
+          xyz="0 0 0"
+          rpy="0 0 0"/>
       <axis xyz="0 1 0"/>
       <dynamics
@@ -350,7 +354,7 @@
     </inertial>
   </link>
-  <!-- Required base_link -> camera_link transform -->
-  <joint name="camera_joint"
-         type="fixed">
+  <joint
+      name="camera_joint"
+      type="fixed">
     <parent link="base_link"/>
     <child link="camera_link"/>
@@ -400,7 +404,7 @@
     </inertial>
   </link>
-  <!-- Required base_link -> laser_link transform -->
-  <joint name="laser_joint"
-         type="fixed">
+  <joint
+      name="laser_joint"
+      type="fixed">
     <parent link="base_link"/>
     <child link="laser_link"/>
@@ -412,22 +416,9 @@
   <!-- GAZEBO VISUAL MATERIALS                                  -->
   <!-- ========================================================= -->
-  <!--
-       Gazebo classic's legacy URDF "gazebo extension" converter
-       expects <material> under <gazebo reference="..."> to be a
-       PLAIN TEXT built-in Ogre material script name (e.g.
-       "Gazebo/Blue"), not nested <ambient>/<diffuse> elements and
-       not wrapped in a named <visual> tag - both of those forms
-       were silently dropped, which is why the model kept
-       rendering grey. Each link below uses one of Gazebo's
-       built-in material names as the closest match to the
-       original custom RGBA colors.
-       Each link also gets exactly ONE <gazebo reference="...">
-       block (material + friction + sensor all merged together).
-       Multiple separate <gazebo reference> blocks for the same
-       link are not guaranteed to merge cleanly in Gazebo classic.
-  -->
+  <!-- Blue chassis -->
   <gazebo reference="base_link">
     <material>Gazebo/Blue</material>
   </gazebo>
+  <!-- Grey steering knuckles -->
   <gazebo reference="front_left_steering_link">
     <material>Gazebo/Grey</material>
@@ -436,4 +427,7 @@
     <material>Gazebo/Grey</material>
   </gazebo>
+  <!-- ========================================================= -->
+  <!-- WHEEL MATERIALS AND CONTACT                              -->
+  <!-- ========================================================= -->
   <gazebo reference="front_left_wheel_link">
     <material>Gazebo/FlatBlack</material>
@@ -465,11 +459,11 @@
   </gazebo>
   <!-- ========================================================= -->
-  <!-- GAZEBO RGB CAMERA (material + sensor merged into ONE      -->
-  <!-- <gazebo reference="camera_link"> block)                  -->
+  <!-- GAZEBO RGB CAMERA                                        -->
   <!-- ========================================================= -->
   <gazebo reference="camera_link">
     <material>Gazebo/DarkGrey</material>
-    <sensor name="front_camera"
-            type="camera">
+    <sensor
+        name="front_camera"
+        type="camera">
       <always_on>true</always_on>
       <update_rate>10.0</update_rate>
@@ -501,24 +495,15 @@
   <!-- GAZEBO 2D LIDAR                                          -->
   <!-- ========================================================= -->
-  <!--
-       This is the ONLY new functional addition relative to the
-       verified camera + controller configuration.
-       Output:
-         /scan
-       Type:
-         sensor_msgs/msg/LaserScan
-       Frame:
-         laser_link
-  -->
   <gazebo reference="laser_link">
     <material>Gazebo/DarkGrey</material>
-    <sensor name="lidar"
-            type="ray">
+    <sensor
+        name="lidar"
+        type="ray">
       <always_on>true</always_on>
       <update_rate>10.0</update_rate>
+      <!-- Keep LiDAR rays visible -->
       <visualize>true</visualize>
       <pose>0 0 0 0 0 0</pose>
       <ray>
-        <!-- 360 degree horizontal scan -->
         <scan>
           <horizontal>
@@ -529,5 +514,4 @@
           </horizontal>
         </scan>
-        <!-- Measurement range -->
         <range>
           <min>0.05</min>
@@ -535,5 +519,4 @@
           <resolution>0.01</resolution>
         </range>
-        <!-- Small Gaussian noise -->
         <noise>
           <type>gaussian</type>
@@ -542,5 +525,4 @@
         </noise>
       </ray>
-      <!-- ROS 2 LaserScan plugin -->
       <plugin
           name="laser_controller"
@@ -558,21 +540,11 @@
   <!-- ROS 2 CONTROL                                            -->
   <!-- ========================================================= -->
-  <!--
-       IMPORTANT:
-       This section is retained in the same form as the verified
-       Milestone 4 / camera-working version.
-  -->
   <ros2_control
       name="GazeboSystem"
       type="system">
-    <!-- ======================================================= -->
-    <!-- HARDWARE PLUGIN                                        -->
-    <!-- ======================================================= -->
     <hardware>
       <plugin>gazebo_ros2_control/GazeboSystem</plugin>
     </hardware>
-    <!-- ======================================================= -->
-    <!-- FRONT LEFT STEERING                                    -->
-    <!-- ======================================================= -->
+    <!-- Front-left steering -->
     <joint name="front_left_steering_joint">
       <command_interface name="position">
@@ -583,7 +555,5 @@
       <state_interface name="velocity"/>
     </joint>
-    <!-- ======================================================= -->
-    <!-- FRONT RIGHT STEERING                                   -->
-    <!-- ======================================================= -->
+    <!-- Front-right steering -->
     <joint name="front_right_steering_joint">
       <command_interface name="position">
@@ -594,7 +564,5 @@
       <state_interface name="velocity"/>
     </joint>
-    <!-- ======================================================= -->
-    <!-- REAR LEFT DRIVE                                        -->
-    <!-- ======================================================= -->
+    <!-- Rear-left drive -->
     <joint name="rear_left_wheel_joint">
       <command_interface name="velocity"/>
@@ -602,7 +570,5 @@
       <state_interface name="velocity"/>
     </joint>
-    <!-- ======================================================= -->
-    <!-- REAR RIGHT DRIVE                                       -->
-    <!-- ======================================================= -->
+    <!-- Rear-right drive -->
     <joint name="rear_right_wheel_joint">
       <command_interface name="velocity"/>
@@ -610,14 +576,10 @@
       <state_interface name="velocity"/>
     </joint>
-    <!-- ======================================================= -->
-    <!-- FRONT LEFT FREE-ROLLING WHEEL                          -->
-    <!-- ======================================================= -->
+    <!-- Front-left free rolling -->
     <joint name="front_left_wheel_joint">
       <state_interface name="position"/>
       <state_interface name="velocity"/>
     </joint>
-    <!-- ======================================================= -->
-    <!-- FRONT RIGHT FREE-ROLLING WHEEL                         -->
-    <!-- ======================================================= -->
+    <!-- Front-right free rolling -->
     <joint name="front_right_wheel_joint">
       <state_interface name="position"/>
@@ -635,3 +597,50 @@
     </plugin>
   </gazebo>
+  <!-- ========================================================= -->
+  <!-- GAZEBO GROUND-TRUTH ODOMETRY                             -->
+  <!-- ========================================================= -->
+  <!--
+       Task 2 trajectory-analysis pose source.
+       IMPORTANT:
+       Gazebo Classic collapses the fixed base_link into
+       base_footprint during URDF -> SDF conversion.
+       Therefore P3D must track base_footprint rather than
+       base_link.
+       Output:
+           /odom
+       Message:
+           nav_msgs/msg/Odometry
+       This is ground-truth simulation data and is intended only
+       for Task 2 model verification / trajectory analysis.
+  -->
+  <gazebo>
+    <plugin
+        name="ground_truth_odometry"
+        filename="libgazebo_ros_p3d.so">
+      <ros>
+        <namespace>/</namespace>
+        <!--
+             The P3D plugin internally publishes "odom".
+             Explicitly remap it to /odom.
+        -->
+        <remapping>odom:=odom</remapping>
+      </ros>
+      <!--
+           Track the Gazebo physics root.
+           Do NOT change this back to base_link unless
+           base_link is explicitly preserved in the generated
+           Gazebo SDF.
+      -->
+      <body_name>base_footprint</body_name>
+      <!-- World-coordinate ground truth -->
+      <frame_name>world</frame_name>
+      <!-- 50 Hz trajectory sampling -->
+      <update_rate>50.0</update_rate>
+      <!-- No artificial pose offsets -->
+      <xyz_offset>0 0 0</xyz_offset>
+      <rpy_offset>0 0 0</rpy_offset>
+      <!-- Ground truth: no measurement noise -->
+      <gaussian_noise>0.0</gaussian_noise>
+    </plugin>
+  </gazebo>
 </robot>

Commit message: Updates for task 2

File: ros2_ws/src/ee5112_vehicle/urdf/vehicle.urdf.xacro (robot description, xacro)
@@ -12,4 +12,5 @@
   <!-- ========================================================= -->
   <xacro:arg name="controllers_file" default=""/>
+  <xacro:arg name="sensor_visuals" default="false"/>
   <!-- ========================================================= -->
   <!-- VEHICLE PARAMETERS                                       -->
@@ -231,6 +232,6 @@
       <axis xyz="0 1 0"/>
       <dynamics
-          damping="0.02"
-          friction="0.01"/>
+          damping="0.00"
+          friction="0.00"/>
     </joint>
   </xacro:macro>
@@ -294,6 +295,7 @@
       <axis xyz="0 1 0"/>
       <dynamics
-          damping="0.02"
-          friction="0.01"/>
+          damping="0.00"
+          friction="0.00"/>
+      <limit effort="5.0" velocity="15.0"/>
     </joint>
   </xacro:macro>
@@ -338,7 +340,31 @@
       <material name="camera_lens_colour"/>
     </visual>
+    <!-- Mounting pedestal: sits ON the chassis top without penetrating it.
+         camera_link is at z=0.08 in base_link, chassis top is at z=0.06
+         (z=-0.02 here), camera body bottom is at z=0.065 (z=-0.015 here).
+         The pedestal spans z=-0.020 (flush on chassis top) to z=-0.014
+         (1 mm hidden inside the camera body). It is inset 5 mm from the
+         chassis front face (x=0.15 in base_link) so no faces are coplanar
+         with the chassis, which avoids z-fighting. -->
+    <visual>
+      <origin
+          xyz="-0.00625 0 -0.017"
+          rpy="0 0 0"/>
+      <geometry>
+        <box size="0.0225 0.040 0.006"/>
+      </geometry>
+      <material name="sensor_dark"/>
+    </visual>
     <collision>
       <geometry>
         <box size="0.035 0.050 0.030"/>
+      </geometry>
+    </collision>
+    <collision>
+      <origin
+          xyz="-0.00625 0 -0.017"
+          rpy="0 0 0"/>
+      <geometry>
+        <box size="0.0225 0.040 0.006"/>
       </geometry>
     </collision>
@@ -375,15 +401,29 @@
       <material name="sensor_dark"/>
     </visual>
+    <!-- Mounting post: laser_link is at z=0.18 above base_link origin,
+         chassis top is at z=0.06, laser body bottom is at z=0.16.
+         In the laser_link frame the post spans z=-0.125 (5 mm sunk into
+         the chassis) to z=-0.02 (bottom of the lidar body). -->
     <visual>
       <origin
-          xyz="0 0 -0.035"
+          xyz="0 0 -0.0725"
           rpy="0 0 0"/>
       <geometry>
         <cylinder
             radius="0.008"
-            length="0.030"/>
+            length="0.105"/>
       </geometry>
       <material name="steering_grey"/>
     </visual>
+    <collision>
+      <origin
+          xyz="0 0 -0.0725"
+          rpy="0 0 0"/>
+      <geometry>
+        <cylinder
+            radius="0.008"
+            length="0.105"/>
+      </geometry>
+    </collision>
     <collision>
       <geometry>
@@ -468,5 +508,5 @@
       <always_on>true</always_on>
       <update_rate>10.0</update_rate>
-      <visualize>true</visualize>
+      <visualize>$(arg sensor_visuals)</visualize>
       <camera name="camera">
         <horizontal_fov>1.3962634</horizontal_fov>
@@ -503,5 +543,5 @@
       <update_rate>10.0</update_rate>
       <!-- Keep LiDAR rays visible -->
-      <visualize>true</visualize>
+      <visualize>$(arg sensor_visuals)</visualize>
       <pose>0 0 0 0 0 0</pose>
       <ray>
